File: nanosaur-exp-board.sch (KiCad schematic (older format))
At the start: 13 parts, among them J1 jetson_nano, J2 Screw_Terminal_01x02, J3 Conn_oled_right, J4 Conn_oled_left, J5 Conn_motors, J6 Conn_01x03, SW1 SW_SPDT

Commit message: Improve sch and pcb
Parts:
- J3: value Conn_oled_right -> Conn_01x04
- J4: value Conn_oled_left -> Conn_01x04
- J5: value Conn_motors -> Conn_01x04
Changed lines of the file:
@@
 P 8200 2350
 F 0 "J3" H 8280 2342 50  0000 L CNN
-F 1 "Conn_oled_right" H 8280 2251 50  0000 L CNN
+F 1 "Conn_01x04" H 8280 2251 50  0000 L CNN
 F 2 "Connector_PinHeader_2.54mm:PinHeader_1x04_P2.54mm_Vertical" H 8200 2350 50  0001 C CNN
 F 3 "~" H 8200 2350 50  0001 C CNN
@@
 P 8200 3000
 F 0 "J4" H 8280 2992 50  0000 L CNN
-F 1 "Conn_oled_left" H 8280 2901 50  0000 L CNN
+F 1 "Conn_01x04" H 8280 2901 50  0000 L CNN
 F 2 "Connector_PinHeader_2.54mm:PinHeader_1x04_P2.54mm_Vertical" H 8200 3000 50  0001 C CNN
 F 3 "~" H 8200 3000 50  0001 C CNN
@@
 P 8200 3650
 F 0 "J5" H 8280 3642 50  0000 L CNN
-F 1 "Conn_motors" H 8280 3551 50  0000 L CNN
+F 1 "Conn_01x04" H 8280 3551 50  0000 L CNN
 F 2 "Connector_PinHeader_2.54mm:PinHeader_1x04_P2.54mm_Vertical" H 8200 3650 50  0001 C CNN
 F 3 "~" H 8200 3650 50  0001 C CNN

Commit message: Improve sch and pcb
Parts:
- removed J5: Conn_01x04, Connector_PinHeader_2.54mm:PinHeader_1x04_P2.54mm_Vertical, symbol Connector_Generic:Conn_01x04
- added H5, H6: MountingHole, MountingHole:MountingHole_2.2mm_M2, symbol Mechanical:MountingHole
- added J5: Conn_01x06, Connector_PinHeader_2.54mm:PinHeader_1x06_P2.54mm_Vertical, symbol Connector_Generic:Conn_01x06
- added J7: Conn_01x04, Connector_PinHeader_2.54mm:PinHeader_1x04_P2.54mm_Vertical, symbol Connector_Generic:Conn_01x04
- H1, H2, H3, H4: footprint MountingHole:MountingHole_2.2mm_M2_ISO7380_Pad -> MountingHole:MountingHole_2.2mm_M2
Connections:
- wire segments 63 -> 73
Other:
- moved on the sheet: J3, J4, J6, R1, R2

Commit message: Improve sch and azz gerber zip
Other:
- note added: "Optional\nI2C"
Changed lines of the file:
@@
 Wire Notes Line
 	7400 3400 7400 2800
+Text Notes 8550 3000 0    50   ~ 0
+Optional\nI2C
 $EndSCHEMATC
