File: nanosaur-exp-board.sch (KiCad schematic (older format))
At the start: 16 parts, among them J1 jetson_nano, J2 Screw_Terminal_01x02, J3 Conn_01x04, J4 Conn_01x04, J5 Conn_01x06, J6 Conn_01x03, J7 Conn_01x04, SW1 SW_SPDT

Commit message: Improve PCB layout, fix BOM, improve sch
Parts:
- removed H1, H2, H3, H4, H5, H6: MountingHole, MountingHole:MountingHole_2.2mm_M2, symbol Mechanical:MountingHole
- J1: footprint Connector_PinSocket_2.54mm:PinSocket_2x21_P2.54mm_Vertical -> Connector_PinSocket_2.54mm:PinSocket_2x20_P2.54mm_Vertical; Component (none) -> PinHeader 2x20 - P2.54mm
- J2: Component (none) -> Terminal block 1x02 - 2.54mm
- J3, J4: value Conn_01x04 -> Conn_i2c_oled; Component (none) -> cable 1x4 length 200mm
- J5: value Conn_01x06 -> Conn_motors; Component (none) -> cable 1x6 length 180mm
- J6: value Conn_01x03 -> Conn_buttons; Component (none) -> cable 1x3 length 220mm
- J7: Component (none) -> Pin Header (optional*)
- R1, R2: Component (none) -> Resistor THT 1/4W
- SW1: Component (none) -> Slide switch P4.7mm
Connections:
- net labels added: MountingHole

Commit message: fix bom
Parts:
- J7: Component Pin Header (optional*) -> Pin Header 1x3 (optional*)
Changed lines of the file:
@@
 F 2 "Connector_PinHeader_2.54mm:PinHeader_1x04_P2.54mm_Vertical" H 8200 3000 50  0001 C CNN
 F 3 "~" H 8200 3000 50  0001 C CNN
-F 4 "Pin Header (optional*)" H 8200 3000 50  0001 C CNN "Component"
+F 4 "Pin Header 1x3 (optional*)" H 8200 3000 50  0001 C CNN "Component"
 	1    8200 3000
 	1    0    0    -1

Commit message: Fix readme
Parts:
- J3, J4: Component cable 1x4 length 200mm -> cable 1x4 length 300mm
- J5: Component cable 1x6 length 180mm -> cable 1x6 length 210mm
- J6: Component cable 1x3 length 220mm -> cable 1x3 length 300mm
- R1, R2: footprint Resistor_THT:R_Axial_DIN0204_L3.6mm_D1.6mm_P7.62mm_Horizontal -> Resistor_THT:R_Axial_DIN0207_L6.3mm_D2.5mm_P10.16mm_Horizontal
Changed lines of the file:
@@
 Title "Expansion board"
 Date ""
-Rev "1"
+Rev "1.1"
 Comp "nanosaur"
 Comment1 "Raffaello Bonghi"
-Comment2 ""
+Comment2 "https://nanosaur.ai/"
 Comment3 ""
 Comment4 ""
@@
 NoConn ~ 5950 3950
 NoConn ~ 5950 4150
-Wire Wire Line
-	5950 2600 6850 2600
-Wire Wire Line
-	5950 2700 6950 2700
 $Comp
 L power:GND #PWR0111
@@
 F 0 "R1" H 7620 4796 50  0000 L CNN
 F 1 "1k" H 7620 4705 50  0000 L CNN
-F 2 "Resistor_THT:R_Axial_DIN0204_L3.6mm_D1.6mm_P7.62mm_Horizontal" V 7480 4750 50  0001 C CNN
+F 2 "Resistor_THT:R_Axial_DIN0207_L6.3mm_D2.5mm_P10.16mm_Horizontal" V 7480 4750 50  0001 C CNN
 F 3 "~" H 7550 4750 50  0001 C CNN
 F 4 "Resistor THT 1/4W" H 7550 4750 50  0001 C CNN "Component"
@@
 F 0 "R2" H 7870 4796 50  0000 L CNN
 F 1 "1k" H 7870 4705 50  0000 L CNN
-F 2 "Resistor_THT:R_Axial_DIN0204_L3.6mm_D1.6mm_P7.62mm_Horizontal" V 7730 4750 50  0001 C CNN
+F 2 "Resistor_THT:R_Axial_DIN0207_L6.3mm_D2.5mm_P10.16mm_Horizontal" V 7730 4750 50  0001 C CNN
 F 3 "~" H 7800 4750 50  0001 C CNN
 F 4 "Resistor THT 1/4W" H 7800 4750 50  0001 C CNN "Component"
@@
 F 2 "Connector_PinHeader_2.54mm:PinHeader_1x03_P2.54mm_Vertical" H 8200 5200 50  0001 C CNN
 F 3 "~" H 8200 5200 50  0001 C CNN
-F 4 "cable 1x3 length 220mm" H 8200 5200 50  0001 C CNN "Component"
+F 4 "cable 1x3 length 300mm" H 8200 5200 50  0001 C CNN "Component"
 	1    8200 5200
 	1    0    0    -1
@@
 F 2 "Connector_PinHeader_2.54mm:PinHeader_1x06_P2.54mm_Vertical" H 8200 3750 50  0001 C CNN
 F 3 "~" H 8200 3750 50  0001 C CNN
-F 4 "cable 1x6 length 180mm" H 8200 3750 50  0001 C CNN "Component"
+F 4 "cable 1x6 length 210mm" H 8200 3750 50  0001 C CNN "Component"
 	1    8200 3750
 	1    0    0    -1
@@
 	1    0    0    -1
 $EndComp
-Wire Wire Line
-	6950 1700 8000 1700
-Wire Wire Line
-	6850 1600 8000 1600
 $Comp
 L Connector_Generic:Conn_01x04 J4
@@
 F 2 "Connector_PinHeader_2.54mm:PinHeader_1x04_P2.54mm_Vertical" H 8200 2350 50  0001 C CNN
 F 3 "~" H 8200 2350 50  0001 C CNN
-F 4 "cable 1x4 length 200mm" H 8200 2350 50  0001 C CNN "Component"
+F 4 "cable 1x4 length 300mm" H 8200 2350 50  0001 C CNN "Component"
 	1    8200 2350
 	1    0    0    -1
@@
 F 2 "Connector_PinHeader_2.54mm:PinHeader_1x04_P2.54mm_Vertical" H 8200 1700 50  0001 C CNN
 F 3 "~" H 8200 1700 50  0001 C CNN
-F 4 "cable 1x4 length 200mm" H 8200 1700 50  0001 C CNN "Component"
+F 4 "cable 1x4 length 300mm" H 8200 1700 50  0001 C CNN "Component"
 	1    8200 1700
 	1    0    0    -1
@@
 Wire Wire Line
 	7150 2350 7150 3000
-Wire Wire Line
-	6950 1700 6950 2700
-Wire Wire Line
-	6850 1600 6850 2600
 $Comp
 L power:+3V3 #PWR0120
@@
 EndData
 $EndBitmap
+Wire Wire Line
+	6950 1700 8000 1700
+Wire Wire Line
+	6850 1600 8000 1600
+Wire Wire Line
+	6950 1700 6950 2700
+Wire Wire Line
+	5950 2700 6950 2700
+Wire Wire Line
+	5950 2600 6850 2600
+Wire Wire Line
+	6850 1600 6850 2600
 $EndSCHEMATC

Commit message: Reference buy url
Parts:
- J1: URL (none) -> https://www.aliexpress.com/item/33036974240.html
- J2: URL (none) -> https://www.aliexpress.com/item/1005001894448937.html
- SW1: URL (none) -> https://www.aliexpress.com/item/32723955831.html
Changed lines of the file:
@@
 F 3 "~" H 1450 2000 50  0001 C CNN
 F 4 "Terminal block 1x02 - 2.54mm" H 1450 2000 50  0001 C CNN "Component"
+F 5 "https://www.aliexpress.com/item/1005001894448937.html" H 1450 2000 50  0001 C CNN "URL"
 	1    1450 2000
 	0    -1   -1   0
@@
 F 3 "~" H 2300 2300 50  0001 C CNN
 F 4 "Slide switch P4.7mm" H 2300 2300 50  0001 C CNN "Component"
+F 5 "https://www.aliexpress.com/item/32723955831.html" H 2300 2300 50  0001 C CNN "URL"
 	1    2300 2300
 	1    0    0    -1
@@
 F 3 "~" H 5300 3250 50  0001 C CNN
 F 4 "PinHeader 2x20 - P2.54mm" H 5050 3550 50  0001 C CNN "Component"
+F 5 "https://www.aliexpress.com/item/33036974240.html" H 5050 3550 50  0001 C CNN "URL"
 	1    5050 3550
 	1    0    0    -1

Commit message: Added other documentation fields
Parts:
- J3, J4, J5, J6: Note (none) -> Read documentation; URL (none) -> https://www.aliexpress.com/item/1005003596191061.html
- R1, R2: Component Resistor THT 1/4W -> Resistor THT 1/4W (optional*); URL (none) -> https://www.aliexpress.com/item/1005003629359182.html
Changed lines of the file:
@@
 F 2 "Resistor_THT:R_Axial_DIN0207_L6.3mm_D2.5mm_P10.16mm_Horizontal" V 7480 4750 50  0001 C CNN
 F 3 "~" H 7550 4750 50  0001 C CNN
-F 4 "Resistor THT 1/4W" H 7550 4750 50  0001 C CNN "Component"
+F 4 "Resistor THT 1/4W (optional*)" H 7550 4750 50  0001 C CNN "Component"
+F 5 "https://www.aliexpress.com/item/1005003629359182.html" H 7550 4750 50  0001 C CNN "URL"
 	1    7550 4750
 	1    0    0    -1
@@
 F 2 "Resistor_THT:R_Axial_DIN0207_L6.3mm_D2.5mm_P10.16mm_Horizontal" V 7730 4750 50  0001 C CNN
 F 3 "~" H 7800 4750 50  0001 C CNN
-F 4 "Resistor THT 1/4W" H 7800 4750 50  0001 C CNN "Component"
+F 4 "Resistor THT 1/4W (optional*)" H 7800 4750 50  0001 C CNN "Component"
+F 5 "https://www.aliexpress.com/item/1005003629359182.html" H 7800 4750 50  0001 C CNN "URL"
 	1    7800 4750
 	1    0    0    -1
@@
 F 3 "~" H 8200 5200 50  0001 C CNN
 F 4 "cable 1x3 length 300mm" H 8200 5200 50  0001 C CNN "Component"
+F 5 "https://www.aliexpress.com/item/1005003596191061.html" H 8200 5200 50  0001 C CNN "URL"
+F 6 "Read documentation" H 8200 5200 50  0001 C CNN "Note"
 	1    8200 5200
 	1    0    0    -1
@@
 F 3 "~" H 8200 3750 50  0001 C CNN
 F 4 "cable 1x6 length 210mm" H 8200 3750 50  0001 C CNN "Component"
+F 5 "https://www.aliexpress.com/item/1005003596191061.html" H 8200 3750 50  0001 C CNN "URL"
+F 6 "Read documentation" H 8200 3750 50  0001 C CNN "Note"
 	1    8200 3750
 	1    0    0    -1
@@
 F 3 "~" H 8200 2350 50  0001 C CNN
 F 4 "cable 1x4 length 300mm" H 8200 2350 50  0001 C CNN "Component"
+F 5 "Read documentation" H 8200 2350 50  0001 C CNN "Note"
+F 6 "https://www.aliexpress.com/item/1005003596191061.html" H 8200 2350 50  0001 C CNN "URL"
 	1    8200 2350
 	1    0    0    -1
@@
 F 3 "~" H 8200 1700 50  0001 C CNN
 F 4 "cable 1x4 length 300mm" H 8200 1700 50  0001 C CNN "Component"
+F 5 "Read documentation" H 8200 1700 50  0001 C CNN "Note"
+F 6 "https://www.aliexpress.com/item/1005003596191061.html" H 8200 1700 50  0001 C CNN "URL"
 	1    8200 1700
 	1    0    0    -1

Commit message: fix table fields
Parts:
- J1: Note (none) -> https://www.aliexpress.com/item/33036974240.html; URL https://www.aliexpress.com/item/33036974240.html -> (none)
- J2: Note (none) -> https://www.aliexpress.com/item/1005001894448937.html; URL https://www.aliexpress.com/item/1005001894448937.html -> (none)
- J3, J4, J5, J6: Note Read documentation -> Read Table connectors; URL https://www.aliexpress.com/item/1005003596191061.html -> (none)
- R1, R2: Note (none) -> https://www.aliexpress.com/item/1005003629359182.html; URL https://www.aliexpress.com/item/1005003629359182.html -> (none)
- SW1: Note (none) -> https://www.aliexpress.com/item/32723955831.html; URL https://www.aliexpress.com/item/32723955831.html -> (none)
Changed lines of the file:
@@
 F 3 "~" H 1450 2000 50  0001 C CNN
 F 4 "Terminal block 1x02 - 2.54mm" H 1450 2000 50  0001 C CNN "Component"
-F 5 "https://www.aliexpress.com/item/1005001894448937.html" H 1450 2000 50  0001 C CNN "URL"
+F 5 "https://www.aliexpress.com/item/1005001894448937.html" H 1450 2000 50  0001 C CNN "Note"
 	1    1450 2000
 	0    -1   -1   0
@@
 F 3 "~" H 2300 2300 50  0001 C CNN
 F 4 "Slide switch P4.7mm" H 2300 2300 50  0001 C CNN "Component"
-F 5 "https://www.aliexpress.com/item/32723955831.html" H 2300 2300 50  0001 C CNN "URL"
+F 5 "https://www.aliexpress.com/item/32723955831.html" H 2300 2300 50  0001 C CNN "Note"
 	1    2300 2300
 	1    0    0    -1
@@
 F 3 "~" H 7550 4750 50  0001 C CNN
 F 4 "Resistor THT 1/4W (optional*)" H 7550 4750 50  0001 C CNN "Component"
-F 5 "https://www.aliexpress.com/item/1005003629359182.html" H 7550 4750 50  0001 C CNN "URL"
+F 5 "https://www.aliexpress.com/item/1005003629359182.html" H 7550 4750 50  0001 C CNN "Note"
 	1    7550 4750
 	1    0    0    -1
@@
 F 3 "~" H 7800 4750 50  0001 C CNN
 F 4 "Resistor THT 1/4W (optional*)" H 7800 4750 50  0001 C CNN "Component"
-F 5 "https://www.aliexpress.com/item/1005003629359182.html" H 7800 4750 50  0001 C CNN "URL"
+F 5 "https://www.aliexpress.com/item/1005003629359182.html" H 7800 4750 50  0001 C CNN "Note"
 	1    7800 4750
 	1    0    0    -1
@@
 F 3 "~" H 8200 5200 50  0001 C CNN
 F 4 "cable 1x3 length 300mm" H 8200 5200 50  0001 C CNN "Component"
-F 5 "https://www.aliexpress.com/item/1005003596191061.html" H 8200 5200 50  0001 C CNN "URL"
-F 6 "Read documentation" H 8200 5200 50  0001 C CNN "Note"
+F 5 "Read Table connectors" H 8200 5200 50  0001 C CNN "Note"
 	1    8200 5200
 	1    0    0    -1
@@
 F 3 "~" H 5300 3250 50  0001 C CNN
 F 4 "PinHeader 2x20 - P2.54mm" H 5050 3550 50  0001 C CNN "Component"
-F 5 "https://www.aliexpress.com/item/33036974240.html" H 5050 3550 50  0001 C CNN "URL"
+F 5 "https://www.aliexpress.com/item/33036974240.html" H 5050 3550 50  0001 C CNN "Note"
 	1    5050 3550
 	1    0    0    -1
@@
 F 3 "~" H 8200 3750 50  0001 C CNN
 F 4 "cable 1x6 length 210mm" H 8200 3750 50  0001 C CNN "Component"
-F 5 "https://www.aliexpress.com/item/1005003596191061.html" H 8200 3750 50  0001 C CNN "URL"
-F 6 "Read documentation" H 8200 3750 50  0001 C CNN "Note"
+F 5 "Read Table connectors" H 8200 3750 50  0001 C CNN "Note"
 	1    8200 3750
 	1    0    0    -1
@@
 F 3 "~" H 8200 2350 50  0001 C CNN
 F 4 "cable 1x4 length 300mm" H 8200 2350 50  0001 C CNN "Component"
-F 5 "Read documentation" H 8200 2350 50  0001 C CNN "Note"
-F 6 "https://www.aliexpress.com/item/1005003596191061.html" H 8200 2350 50  0001 C CNN "URL"
+F 5 "Read Table connectors" H 8200 2350 50  0001 C CNN "Note"
 	1    8200 2350
 	1    0    0    -1
@@
 F 3 "~" H 8200 1700 50  0001 C CNN
 F 4 "cable 1x4 length 300mm" H 8200 1700 50  0001 C CNN "Component"
-F 5 "Read documentation" H 8200 1700 50  0001 C CNN "Note"
-F 6 "https://www.aliexpress.com/item/1005003596191061.html" H 8200 1700 50  0001 C CNN "URL"
+F 5 "Read Table connectors" H 8200 1700 50  0001 C CNN "Note"
 	1    8200 1700
 	1    0    0    -1
