File: nanosaur-exp-board.kicad_pcb (KiCad board)
At the start: 2 copper layers, 80 x 20 mm, 21 parts, among them J1 jetson_nano, J2 Screw_Terminal_01x02, J3 Conn_i2c_oled, J4 Conn_i2c_oled, J5 Conn_motors, J6 Conn_buttons, J7 Conn_01x04, SW1 SW_SPDT

Commit message: Final PCB fix
Routing:
- net GND: vias 0 -> 3

Commit message: Fix license and minor fixes
Parts:
- removed the G*** at (111.3, 91.8)
- added G***: LOGO, nanosaur:pizzarobotics, B.Cu at (111.8, 92.9)

Commit message: Fix readme
Parts:
- R1, R2: footprint Resistor_THT:R_Axial_DIN0204_L3.6mm_D1.6mm_P7.62mm_Horizontal -> Resistor_THT:R_Axial_DIN0207_L6.3mm_D2.5mm_P10.16mm_Horizontal
- moved R2 0.90 mm to (137.1, 95.5)
Routing:
- net Net-(J1-Pad31): track 15.1 -> 13.8 mm
- net GND: vias 3 -> 2
Other:
- board text added: "v1.1"
- board text removed: "v1.0"

Commit message: Fix DRC
Parts:
- moved R1 0.12 mm to (136.9, 92.4)
- moved R2 0.10 mm to (137.0, 95.5)
